File: BBB_Rev2/BBB_Cape.brd (EAGLE design)
At the start: 100 x 80 mm, 12 parts, among them SW1 SPST_TACT-EVQQ2

Commit message: updated Cape schematic, added BOM
Parts:
- R1, R2, R3, R4: value 820 -> 330
Changed lines of the file:
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@@
 </autorouter>
 <elements>
-<element name="U$1" library="adafruit" package="BEAGLEBONE_SHIELD" value="BEAGLEBONE_OUTLINE" x="7.62" y="58.42" smashed="yes" rot="R270"/>
-<element name="R1" library="adafruit" package="R0805" value="820" x="30.48" y="48.26" smashed="yes" rot="R270">
+<element name="U$1" library="adafruit" package="BEAGLEBONE_SHIELD" value="BEAGLEBONE_OUTLINE" x="7.62" y="58.42" smashed="yes" rot="R270">
+<attribute name="OC_NEWARK" value="unknown" x="7.62" y="58.42" size="1.778" layer="27" rot="R270" display="off"/>
+<attribute name="MF" value="" x="7.62" y="58.42" size="1.778" layer="27" rot="R270" display="off"/>
+<attribute name="MPN" value="" x="7.62" y="58.42" size="1.778" layer="27" rot="R270" display="off"/>
+</element>
+<element name="R1" library="adafruit" package="R0805" value="330" x="30.48" y="48.26" smashed="yes" rot="R270">
 <attribute name="NAME" x="31.496" y="49.022" size="0.6096" layer="25" rot="R270"/>
+<attribute name="OC_NEWARK" value="02J2330" x="30.48" y="48.26" size="1.778" layer="27" rot="R270" display="off"/>
+<attribute name="MF" value="BOURNS, INC." x="30.48" y="48.26" size="1.778" layer="27" rot="R270" display="off"/>
+<attribute name="MPN" value="CR0603-JW-331ELF" x="30.48" y="48.26" size="1.778" layer="27" rot="R270" display="off"/>
 </element>
-<element name="R2" library="adafruit" package="R0805" value="820" x="33.02" y="48.26" smashed="yes" rot="R270">
+<element name="R2" library="adafruit" package="R0805" value="330" x="33.02" y="48.26" smashed="yes" rot="R270">
 <attribute name="NAME" x="34.036" y="49.022" size="0.6096" layer="25" rot="R270"/>
+<attribute name="OC_NEWARK" value="02J2330" x="33.02" y="48.26" size="1.778" layer="27" rot="R270" display="off"/>
+<attribute name="MF" value="BOURNS, INC." x="33.02" y="48.26" size="1.778" layer="27" rot="R270" display="off"/>
+<attribute name="MPN" value="CR0603-JW-331ELF" x="33.02" y="48.26" size="1.778" layer="27" rot="R270" display="off"/>
 </element>
-<element name="R3" library="adafruit" package="R0805" value="820" x="35.56" y="48.26" smashed="yes" rot="R270">
+<element name="R3" library="adafruit" package="R0805" value="330" x="35.56" y="48.26" smashed="yes" rot="R270">
 <attribute name="NAME" x="36.576" y="49.022" size="0.6096" layer="25" rot="R270"/>
+<attribute name="OC_NEWARK" value="02J2330" x="35.56" y="48.26" size="1.778" layer="27" rot="R270" display="off"/>
+<attribute name="MF" value="BOURNS, INC." x="35.56" y="48.26" size="1.778" layer="27" rot="R270" display="off"/>
+<attribute name="MPN" value="CR0603-JW-331ELF" x="35.56" y="48.26" size="1.778" layer="27" rot="R270" display="off"/>
 </element>
 <element name="LED1" library="adafruit" package="CHIPLED_0805" value="Red" x="30.48" y="43.18" smashed="yes" rot="R180">
 <attribute name="NAME" x="31.75" y="44.45" size="0.6096" layer="25" rot="R270" align="center-left"/>
+<attribute name="OC_NEWARK" value="96W6960" x="30.48" y="43.18" size="1.778" layer="27" rot="R180" display="off"/>
+<attribute name="MF" value="" x="30.48" y="43.18" size="1.778" layer="27" rot="R180" display="off"/>
+<attribute name="MPN" value="KPT-2012SECK-J3" x="30.48" y="43.18" size="1.778" layer="27" rot="R180" display="off"/>
 </element>
 <element name="LED2" library="adafruit" package="CHIPLED_0805" value="Orange" x="33.02" y="43.18" smashed="yes" rot="R180">
 <attribute name="NAME" x="34.29" y="44.45" size="0.6096" layer="25" rot="R270" align="center-left"/>
+<attribute name="OC_NEWARK" value="66W1930" x="33.02" y="43.18" size="1.778" layer="27" rot="R180" display="off"/>
+<attribute name="MF" value="" x="33.02" y="43.18" size="1.778" layer="27" rot="R180" display="off"/>
+<attribute name="MPN" value="KP-2012SECK" x="33.02" y="43.18" size="1.778" layer="27" rot="R180" display="off"/>
 </element>
 <element name="LED3" library="adafruit" package="CHIPLED_0805" value="Green" x="35.56" y="43.18" smashed="yes" rot="R180">
 <attribute name="NAME" x="36.83" y="44.45" size="0.6096" layer="25" rot="R270" align="center-left"/>
+<attribute name="OC_NEWARK" value="66W1927" x="35.56" y="43.18" size="1.778" layer="27" rot="R180" display="off"/>
+<attribute name="MF" value="" x="35.56" y="43.18" size="1.778" layer="27" rot="R180" display="off"/>
+<attribute name="MPN" value="KP-2012CGCK" x="35.56" y="43.18" size="1.778" layer="27" rot="R180" display="off"/>
 </element>
-<element name="U$2" library="quad" package="EM" value="EM_BLUETOOTH" x="77.47" y="45.72" smashed="yes" rot="R180"/>
-<element name="R4" library="adafruit" package="R0805" value="820" x="29.21" y="12.7" smashed="yes" rot="R90">
+<element name="U$2" library="quad" package="EM" value="EM_BLUETOOTH" x="77.47" y="45.72" smashed="yes" rot="R180">
+<attribute name="OC_NEWARK" value="unknown" x="77.47" y="45.72" size="1.778" layer="27" rot="R180" display="off"/>
+<attribute name="MF" value="" x="77.47" y="45.72" size="1.778" layer="27" rot="R180" display="off"/>
+<attribute name="MPN" value="" x="77.47" y="45.72" size="1.778" layer="27" rot="R180" display="off"/>
+</element>
+<element name="R4" library="adafruit" package="R0805" value="330" x="29.21" y="12.7" smashed="yes" rot="R90">
 <attribute name="NAME" x="29.464" y="15.113" size="0.8128" layer="25" rot="R90"/>
+<attribute name="OC_NEWARK" value="02J2330" x="29.21" y="12.7" size="1.778" layer="27" rot="R90" display="off"/>
+<attribute name="MF" value="BOURNS, INC." x="29.21" y="12.7" size="1.778" layer="27" rot="R90" display="off"/>
+<attribute name="MPN" value="CR0603-JW-331ELF" x="29.21" y="12.7" size="1.778" layer="27" rot="R90" display="off"/>
 </element>
 <element name="LED4" library="adafruit" package="CHIPLED_0805" value="Blue" x="26.67" y="12.7" smashed="yes" rot="R180">
 <attribute name="NAME" x="24.765" y="13.97" size="0.8128" layer="25" rot="R270"/>
+<attribute name="OC_NEWARK" value="49P5362" x="26.67" y="12.7" size="1.778" layer="27" rot="R180" display="off"/>
+<attribute name="MF" value="" x="26.67" y="12.7" size="1.778" layer="27" rot="R180" display="off"/>
+<attribute name="MPN" value="KPHBM-2012PBASURKC" x="26.67" y="12.7" size="1.778" layer="27" rot="R180" display="off"/>
 </element>
 <element name="SW1" library="adafruit" package="EVQ-Q2" value="SPST_TACT-EVQQ2" x="34.29" y="30.48" smashed="yes">
 <attribute name="NAME" x="31.29" y="33.98" size="0.6096" layer="25"/>
+<attribute name="OC_NEWARK" value="unknown" x="34.29" y="30.48" size="1.778" layer="27" display="off"/>
+<attribute name="MF" value="" x="34.29" y="30.48" size="1.778" layer="27" display="off"/>
+<attribute name="MPN" value="" x="34.29" y="30.48" size="1.778" layer="27" display="off"/>
 </element>
 <element name="R5" library="adafruit" package="R0805" value="10k" x="30.48" y="38.1" smashed="yes" rot="R270">
 <attribute name="NAME" x="32.131" y="38.227" size="0.6096" layer="25" rot="R270" align="center"/>
+<attribute name="OC_NEWARK" value="05F1511" x="30.48" y="38.1" size="1.778" layer="27" rot="R270" display="off"/>
+<attribute name="MF" value="VISHAY/DALE" x="30.48" y="38.1" size="1.778" layer="27" rot="R270" display="off"/>
+<attribute name="MPN" value="CRCW080510K0FKTA" x="30.48" y="38.1" size="1.778" layer="27" rot="R270" display="off"/>
 </element>
 </elements>
